File: Hardware/Kicad_Project/EV Meter.kicad_pcb (KiCad board)
At the start: 2 copper layers, 50 x 30 mm, 53 parts, among them SW1 PWRSW, Y1 8M

Commit message: Update PCB gerber
Parts:
- added C5: 104, Capacitor_SMD:C_0603_1608Metric, B.Cu at (149.0, 120.0)
- added EEPROM1: M24C02-FMN, Package_SO:SOIC-8_3.9x4.9mm_P1.27mm, B.Cu at (153.7, 121.3)
- moved R8 8.39 mm to (141.8, 115.0), turned to 180 degrees
- moved R6 7.96 mm to (141.8, 113.1), turned to 180 degrees
- moved R4 7.38 mm to (141.9, 116.8), turned to 180 degrees
- moved G*** 1.07 mm to (153.8, 127.5)
- moved REF** 0.36 mm to (142.7, 107.9)
- renumbered LED to D1, SW1 to PowerSW1, HW_RST to RST1, RL to R_LED1, Rp to R_Prog1, STLINK1 to ST-LINK1, MicroUSB to USB-micro1
Routing:
- net /I2C1_SCL: track 26.7 -> 45.9 mm, vias 2 -> 3
- net /I2C1_SDA: track 24.4 -> 36.9 mm, vias 3 -> 4
- net GND: track 265.3 -> 277.3 mm, vias 8 -> 10
- net VCC: track 110.6 -> 118.7 mm, vias 5 -> 7
- net /KEY0: track 26.3 -> 29.1 mm, vias 2 -> 1
- net /KEY2: track 30.5 -> 31.4 mm, vias 2 -> 1
- net /KEY1: track 25.6 -> 26.0 mm, vias 2 -> 1
Other:
- board text added: "CopyRight@Emoe-studio-Floydfish 2020.3"
- board text removed: "CopyRight @ Emoe-studio->Floydfish 2020.3"
